Commit message: added material names

File: src/robot_description/urdf/ur5.urdf.xacro (robot description, xacro)
@@ -201,5 +201,5 @@
         <mesh filename="package://robot_description/meshes/visual/robotiq_arg2f_base_link.stl"/>
       </geometry>
-      <material name="">
+      <material name="grey">
         <color rgba="0.1 0.1 0.1 1"/>
       </material>
@@ -223,5 +223,5 @@
         <mesh filename="package://robot_description/meshes/visual/robotiq_arg2f_140_outer_knuckle.stl"/>
       </geometry>
-      <material name="">
+      <material name="light_blue">
         <color rgba="0.792156862745098 0.819607843137255 0.933333333333333 1"/>
       </material>
@@ -245,5 +245,5 @@
         <mesh filename="package://robot_description/meshes/visual/robotiq_arg2f_140_outer_finger.stl"/>
       </geometry>
-      <material name="">
+      <material name="grey">
         <color rgba="0.1 0.1 0.1 1"/>
       </material>
@@ -267,5 +267,5 @@
         <mesh filename="package://robot_description/meshes/visual/robotiq_arg2f_140_inner_finger.stl"/>
       </geometry>
-      <material name="">
+      <material name="grey">
         <color rgba="0.1 0.1 0.1 1"/>
       </material>
@@ -284,5 +284,5 @@
         <box size="0.027 0.065 0.0075"/>
       </geometry>
-      <material name="">
+      <material name="light_grey">
         <color rgba="0.9 0.9 0.9 1"/>
       </material>
@@ -293,5 +293,5 @@
         <box size="0.03 0.07 0.0075"/>
       </geometry>
-      <material name="">
+      <material name="light_grey">
         <color rgba="0.9 0.0 0.0 1"/>
       </material>
@@ -309,5 +309,5 @@
         <mesh filename="package://robot_description/meshes/visual/robotiq_arg2f_140_inner_knuckle.stl"/>
       </geometry>
-      <material name="">
+      <material name="grey">
         <color rgba="0.1 0.1 0.1 1"/>
       </material>
@@ -331,5 +331,5 @@
         <mesh filename="package://robot_description/meshes/visual/robotiq_arg2f_140_outer_knuckle.stl"/>
       </geometry>
-      <material name="">
+      <material name="light_blue">
         <color rgba="0.792156862745098 0.819607843137255 0.933333333333333 1"/>
       </material>
@@ -353,5 +353,5 @@
         <mesh filename="package://robot_description/meshes/visual/robotiq_arg2f_140_outer_finger.stl"/>
       </geometry>
-      <material name="">
+      <material name="grey">
         <color rgba="0.1 0.1 0.1 1"/>
       </material>
@@ -375,5 +375,5 @@
         <mesh filename="package://robot_description/meshes/visual/robotiq_arg2f_140_inner_finger.stl"/>
       </geometry>
-      <material name="">
+      <material name="grey">
         <color rgba="0.1 0.1 0.1 1"/>
       </material>
@@ -392,5 +392,5 @@
         <box size="0.027 0.065 0.0075"/>
       </geometry>
-      <material name="">
+      <material name="light_grey">
         <color rgba="0.9 0.9 0.9 1"/>
       </material>
@@ -401,6 +401,6 @@
         <box size="0.03 0.07 0.0075"/>
       </geometry>
-      <material name="">
-        <color rgba="0.9 0.0 0.0 1"/>
+      <material name="red">
+        <color rgba="0.9 0.0 0.0 1.0"/>
       </material>
     </collision>
@@ -417,5 +417,5 @@
         <mesh filename="package://robot_description/meshes/visual/robotiq_arg2f_140_inner_knuckle.stl"/>
       </geometry>
-      <material name="">
+      <material name="grey">
         <color rgba="0.1 0.1 0.1 1"/>
       </material>
